File: Hardware/SparkFun-74HC4051-8-Channel-Mux-Breakout.brd (EAGLE design)
At the start: 12.7 x 27.9 mm, 14 parts, among them U1 74HC4051BQ

Commit message: Used improved SparkFun libraries to remove the need for separate library. Removed single part library. Resolves #3
Parts:
- U1: value 74HC4051BQ -> (none); device 8mux:DHVQFN-16-2.5X3.5MM -> SparkFun-IC-Logic:DHVQFN-16-2.5X3.5MM
Changed lines of the file:
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@@
 <?xml version="1.0" encoding="utf-8"?>
 <!DOCTYPE eagle SYSTEM "eagle.dtd">
-<eagle version="7.5.0">
+<eagle version="7.7.0">
 <drawing>
 <settings>
@@
 <attribute name="PROD_ID" value="CONN-08437" x="1.27" y="6.35" size="1.778" layer="28" rot="MR90" display="off"/>
 </element>
-<element name="U1" library="8mux" package="DHVQFN-16-2.5X3.5MM" value="74HC4051BQ" x="6.35" y="13.97" rot="R270">
+<element name="U1" library="SparkFun-IC-Logic" package="DHVQFN-16-2.5X3.5MM" value="" x="6.35" y="13.97" rot="R270">
 <attribute name="PROD_ID" value="IC-13334" x="6.35" y="13.97" size="1.778" layer="27" rot="R270" display="off"/>
 </element>
